File: neon/neon.sch (KiCad schematic (older format))
At the start: 41 parts, among them J1 VBUS-VCC, J2 V3V3-GND, J3 V3V3-GND, J4 V3V3-GND, J5 V3V3-VIO, Q1 BC807, Q2 BC807, Q3 BC807, Q4 BC807, Q5 BC807, Q6 BC807, Q7 BC807, Q8 BC807, U2 CBUS, U3 DBUS, U4 ABUS, U5 BBUS

Commit message: Assign footprints - part 1 and buggy
Parts:
- D1, D2, D3, D4, D5, D6, D7, D8: footprint (none) -> LED_SMD:LED_0805_2012Metric
- J1, J2, J3, J4, J5: footprint (none) -> Connector_PinHeader_2.54mm:PinHeader_1x02_P2.54mm_Vertical
- R1, R10, R11, R12, R13, R14, R15, R16, R2, R3, R4, R5, R6, R7, R8, R9: footprint (none) -> Resistor_SMD:R_0805_2012Metric
- U2, U3, U4, U5: footprint (none) -> Connector_PinHeader_2.54mm:PinHeader_1x08_P2.54mm_Vertical
Changed lines of the file:
@@
 F 0 "U3" H 3850 3800 50  0000 C CNN
 F 1 "DBUS" H 3900 3700 50  0000 C CNN
-F 2 "" H 3375 4475 50  0001 C CNN
+F 2 "Connector_PinHeader_2.54mm:PinHeader_1x08_P2.54mm_Vertical" H 3375 4475 50  0001 C CNN
 F 3 "" H 3375 4475 50  0001 C CNN
 	1    3400 3800
@@
 F 0 "J2" V 5800 5150 50  0000 L CNN
 F 1 "V3V3-GND" H 5600 5100 50  0001 C CNN
-F 2 "" H 5600 5300 50  0001 C CNN
+F 2 "Connector_PinHeader_2.54mm:PinHeader_1x02_P2.54mm_Vertical" H 5600 5300 50  0001 C CNN
 F 3 "~" H 5600 5300 50  0001 C CNN
 	1    5600 5300
@@
 F 0 "J3" V 5800 5600 50  0000 L CNN
 F 1 "V3V3-GND" H 5600 5550 50  0001 C CNN
-F 2 "" H 5600 5750 50  0001 C CNN
+F 2 "Connector_PinHeader_2.54mm:PinHeader_1x02_P2.54mm_Vertical" H 5600 5750 50  0001 C CNN
 F 3 "~" H 5600 5750 50  0001 C CNN
 	1    5600 5750
@@
 F 0 "J4" V 5800 6050 50  0000 L CNN
 F 1 "V3V3-GND" H 5600 6000 50  0001 C CNN
-F 2 "" H 5600 6200 50  0001 C CNN
+F 2 "Connector_PinHeader_2.54mm:PinHeader_1x02_P2.54mm_Vertical" H 5600 6200 50  0001 C CNN
 F 3 "~" H 5600 6200 50  0001 C CNN
 	1    5600 6200
@@
 F 0 "J1" H 4550 4750 50  0000 L CNN
 F 1 "VBUS-VCC" H 4650 4450 50  0001 C CNN
-F 2 "" H 4500 4650 50  0001 C CNN
+F 2 "Connector_PinHeader_2.54mm:PinHeader_1x02_P2.54mm_Vertical" H 4500 4650 50  0001 C CNN
 F 3 "~" H 4500 4650 50  0001 C CNN
 	1    4500 4650
@@
 F 0 "U2" H 3850 2750 50  0000 C CNN
 F 1 "CBUS" H 3900 2650 50  0000 C CNN
-F 2 "" H 3375 3425 50  0001 C CNN
+F 2 "Connector_PinHeader_2.54mm:PinHeader_1x08_P2.54mm_Vertical" H 3375 3425 50  0001 C CNN
 F 3 "" H 3375 3425 50  0001 C CNN
 	1    3400 2750
@@
 F 0 "R9" V 8300 1300 50  0000 C CNN
 F 1 "10k" V 8084 1300 50  0000 C CNN
-F 2 "" V 8130 1300 50  0001 C CNN
+F 2 "Resistor_SMD:R_0805_2012Metric" V 8130 1300 50  0001 C CNN
 F 3 "~" H 8200 1300 50  0001 C CNN
 	1    8200 1300
@@
 F 0 "D6" H 9043 1967 50  0000 C CNN
 F 1 "LED" H 9043 1876 50  0000 C CNN
-F 2 "" H 9050 1750 50  0001 C CNN
+F 2 "LED_SMD:LED_0805_2012Metric" H 9050 1750 50  0001 C CNN
 F 3 "~" H 9050 1750 50  0001 C CNN
 	1    9050 1750
@@
 F 0 "R10" V 8300 2050 50  0000 C CNN
 F 1 "10k" V 8084 2050 50  0000 C CNN
-F 2 "" V 8130 2050 50  0001 C CNN
+F 2 "Resistor_SMD:R_0805_2012Metric" V 8130 2050 50  0001 C CNN
 F 3 "~" H 8200 2050 50  0001 C CNN
 	1    8200 2050
@@
 F 0 "D5" H 9043 1217 50  0000 C CNN
 F 1 "LED" H 9043 1126 50  0000 C CNN
-F 2 "" H 9050 1000 50  0001 C CNN
+F 2 "LED_SMD:LED_0805_2012Metric" H 9050 1000 50  0001 C CNN
 F 3 "~" H 9050 1000 50  0001 C CNN
 	1    9050 1000
@@
 F 0 "R5" V 3400 1300 50  0000 C CNN
 F 1 "10k" V 3184 1300 50  0000 C CNN
-F 2 "" V 3230 1300 50  0001 C CNN
+F 2 "Resistor_SMD:R_0805_2012Metric" V 3230 1300 50  0001 C CNN
 F 3 "~" H 3300 1300 50  0001 C CNN
 	1    3300 1300
@@
 F 0 "D2" H 2443 1967 50  0000 C CNN
 F 1 "LED" H 2443 1876 50  0000 C CNN
-F 2 "" H 2450 1750 50  0001 C CNN
+F 2 "LED_SMD:LED_0805_2012Metric" H 2450 1750 50  0001 C CNN
 F 3 "~" H 2450 1750 50  0001 C CNN
 	1    2450 1750
@@
 F 0 "R6" V 3400 2050 50  0000 C CNN
 F 1 "10k" V 3184 2050 50  0000 C CNN
-F 2 "" V 3230 2050 50  0001 C CNN
+F 2 "Resistor_SMD:R_0805_2012Metric" V 3230 2050 50  0001 C CNN
 F 3 "~" H 3300 2050 50  0001 C CNN
 	1    3300 2050
@@
 F 0 "D1" H 2443 1217 50  0000 C CNN
 F 1 "LED" H 2443 1126 50  0000 C CNN
-F 2 "" H 2450 1000 50  0001 C CNN
+F 2 "LED_SMD:LED_0805_2012Metric" H 2450 1000 50  0001 C CNN
 F 3 "~" H 2450 1000 50  0001 C CNN
 	1    2450 1000
@@
 F 0 "R8" V 3400 5350 50  0000 C CNN
 F 1 "10k" V 3184 5350 50  0000 C CNN
-F 2 "" V 3230 5350 50  0001 C CNN
+F 2 "Resistor_SMD:R_0805_2012Metric" V 3230 5350 50  0001 C CNN
 F 3 "~" H 3300 5350 50  0001 C CNN
 	1    3300 5350
@@
 F 0 "D3" H 2443 5117 50  0000 C CNN
 F 1 "LED" H 2443 5026 50  0000 C CNN
-F 2 "" H 2450 4900 50  0001 C CNN
+F 2 "LED_SMD:LED_0805_2012Metric" H 2450 4900 50  0001 C CNN
 F 3 "~" H 2450 4900 50  0001 C CNN
 	1    2450 4900
@@
 F 0 "R7" V 3400 4600 50  0000 C CNN
 F 1 "10k" V 3184 4600 50  0000 C CNN
-F 2 "" V 3230 4600 50  0001 C CNN
+F 2 "Resistor_SMD:R_0805_2012Metric" V 3230 4600 50  0001 C CNN
 F 3 "~" H 3300 4600 50  0001 C CNN
 	1    3300 4600
@@
 F 0 "D4" H 2443 5867 50  0000 C CNN
 F 1 "LED" H 2443 5776 50  0000 C CNN
-F 2 "" H 2450 5650 50  0001 C CNN
+F 2 "LED_SMD:LED_0805_2012Metric" H 2450 5650 50  0001 C CNN
 F 3 "~" H 2450 5650 50  0001 C CNN
 	1    2450 5650
@@
 F 0 "J5" H 6850 4750 50  0000 L CNN
 F 1 "V3V3-VIO" H 6950 4450 50  0001 C CNN
-F 2 "" H 6950 4650 50  0001 C CNN
+F 2 "Connector_PinHeader_2.54mm:PinHeader_1x02_P2.54mm_Vertical" H 6950 4650 50  0001 C CNN
 F 3 "~" H 6950 4650 50  0001 C CNN
 	1    6950 4650
@@
 F 0 "U4" H 8550 2750 50  0000 C CNN
 F 1 "ABUS" H 8600 2650 50  0000 C CNN
-F 2 "" H 8075 3425 50  0001 C CNN
+F 2 "Connector_PinHeader_2.54mm:PinHeader_1x08_P2.54mm_Vertical" H 8075 3425 50  0001 C CNN
 F 3 "" H 8075 3425 50  0001 C CNN
 	1    8100 2750
@@
 F 0 "U5" H 8478 3801 50  0000 L CNN
 F 1 "BBUS" H 8478 3710 50  0000 L CNN
-F 2 "" H 8075 4475 50  0001 C CNN
+F 2 "Connector_PinHeader_2.54mm:PinHeader_1x08_P2.54mm_Vertical" H 8075 4475 50  0001 C CNN
 F 3 "" H 8075 4475 50  0001 C CNN
 	1    8100 3800
@@
 F 0 "R16" V 9400 5550 50  0000 L CNN
 F 1 "330" V 9600 5550 50  0000 L CNN
-F 2 "" V 9430 5650 50  0001 C CNN
+F 2 "Resistor_SMD:R_0805_2012Metric" V 9430 5650 50  0001 C CNN
 F 3 "~" H 9500 5650 50  0001 C CNN
 	1    9500 5650
@@
 F 0 "D8" H 9043 5867 50  0000 C CNN
 F 1 "LED" H 9043 5776 50  0000 C CNN
-F 2 "" H 9050 5650 50  0001 C CNN
+F 2 "LED_SMD:LED_0805_2012Metric" H 9050 5650 50  0001 C CNN
 F 3 "~" H 9050 5650 50  0001 C CNN
 	1    9050 5650
@@
 F 0 "R11" V 8300 4600 50  0000 C CNN
 F 1 "10k" V 8084 4600 50  0000 C CNN
-F 2 "" V 8130 4600 50  0001 C CNN
+F 2 "Resistor_SMD:R_0805_2012Metric" V 8130 4600 50  0001 C CNN
 F 3 "~" H 8200 4600 50  0001 C CNN
 	1    8200 4600
@@
 F 0 "D7" H 9043 5117 50  0000 C CNN
 F 1 "LED" H 9043 5026 50  0000 C CNN
-F 2 "" H 9050 4900 50  0001 C CNN
+F 2 "LED_SMD:LED_0805_2012Metric" H 9050 4900 50  0001 C CNN
 F 3 "~" H 9050 4900 50  0001 C CNN
 	1    9050 4900
@@
 F 0 "R12" V 8300 5350 50  0000 C CNN
 F 1 "10k" V 8084 5350 50  0000 C CNN
-F 2 "" V 8130 5350 50  0001 C CNN
+F 2 "Resistor_SMD:R_0805_2012Metric" V 8130 5350 50  0001 C CNN
 F 3 "~" H 8200 5350 50  0001 C CNN
 	1    8200 5350
@@
 F 0 "R15" V 9400 4800 50  0000 L CNN
 F 1 "330" V 9600 4800 50  0000 L CNN
-F 2 "" V 9430 4900 50  0001 C CNN
+F 2 "Resistor_SMD:R_0805_2012Metric" V 9430 4900 50  0001 C CNN
 F 3 "~" H 9500 4900 50  0001 C CNN
 	1    9500 4900
@@
 F 0 "R14" V 9400 1650 50  0000 L CNN
 F 1 "330" V 9600 1650 50  0000 L CNN
-F 2 "" V 9430 1750 50  0001 C CNN
+F 2 "Resistor_SMD:R_0805_2012Metric" V 9430 1750 50  0001 C CNN
 F 3 "~" H 9500 1750 50  0001 C CNN
 	1    9500 1750
@@
 F 0 "R13" V 9400 900 50  0000 L CNN
 F 1 "330" V 9600 900 50  0000 L CNN
-F 2 "" V 9430 1000 50  0001 C CNN
+F 2 "Resistor_SMD:R_0805_2012Metric" V 9430 1000 50  0001 C CNN
 F 3 "~" H 9500 1000 50  0001 C CNN
 	1    9500 1000
@@
 F 0 "R1" V 1900 900 50  0000 L CNN
 F 1 "330" V 2100 900 50  0000 L CNN
-F 2 "" V 1930 1000 50  0001 C CNN
+F 2 "Resistor_SMD:R_0805_2012Metric" V 1930 1000 50  0001 C CNN
 F 3 "~" H 2000 1000 50  0001 C CNN
 	1    2000 1000
@@
 F 0 "R2" V 1900 1650 50  0000 L CNN
 F 1 "330" V 2100 1650 50  0000 L CNN
-F 2 "" V 1930 1750 50  0001 C CNN
+F 2 "Resistor_SMD:R_0805_2012Metric" V 1930 1750 50  0001 C CNN
 F 3 "~" H 2000 1750 50  0001 C CNN
 	1    2000 1750
@@
 F 0 "R3" V 1900 4800 50  0000 L CNN
 F 1 "330" V 2100 4800 50  0000 L CNN
-F 2 "" V 1930 4900 50  0001 C CNN
+F 2 "Resistor_SMD:R_0805_2012Metric" V 1930 4900 50  0001 C CNN
 F 3 "~" H 2000 4900 50  0001 C CNN
 	1    2000 4900
@@
 F 0 "R4" V 1900 5550 50  0000 L CNN
 F 1 "330" V 2100 5550 50  0000 L CNN
-F 2 "" V 1930 5650 50  0001 C CNN
+F 2 "Resistor_SMD:R_0805_2012Metric" V 1930 5650 50  0001 C CNN
 F 3 "~" H 2000 5650 50  0001 C CNN
 	1    2000 5650

Commit message: Pin warning fixes
Changed lines of the file:
@@
 	0    1    1    0
 $EndComp
+$Comp
+L power:PWR_FLAG #FLG0101
+U 1 1 5F61B8EB
+P 9800 3300
+F 0 "#FLG0101" H 9800 3375 50  0001 C CNN
+F 1 "PWR_FLAG" H 9800 3473 50  0000 C CNN
+F 2 "" H 9800 3300 50  0001 C CNN
+F 3 "~" H 9800 3300 50  0001 C CNN
+	1    9800 3300
+	1    0    0    -1
+$EndComp
+$Comp
+L power:GND #PWR0102
+U 1 1 5F61BEF4
+P 9800 3300
+F 0 "#PWR0102" H 9800 3050 50  0001 C CNN
+F 1 "GND" H 9805 3127 50  0000 C CNN
+F 2 "" H 9800 3300 50  0001 C CNN
+F 3 "" H 9800 3300 50  0001 C CNN
+	1    9800 3300
+	1    0    0    -1
+$EndComp
 $EndSCHEMATC

Commit message: Order pins on footprint - part 2
Parts:
- renumbered U4 to A, U5 to B, U2 to C, U3 to D
Changed lines of the file:
@@
 $EndDescr
 $Comp
-L FTDI:DBUS U3
+L FTDI:DBUS D
 U 1 1 5F52AE75
 P 3400 3800
-F 0 "U3" H 3850 3800 50  0000 C CNN
+F 0 "D" H 3850 3800 50  0000 C CNN
 F 1 "DBUS" H 3900 3700 50  0000 C CNN
 F 2 "Connector_PinHeader_2.54mm:PinHeader_1x08_P2.54mm_Vertical" H 3375 4475 50  0001 C CNN
@@
 	5150 2650 3600 2650
 $Comp
-L FTDI:CBUS U2
+L FTDI:CBUS C
 U 1 1 5F520AE1
 P 3400 2750
-F 0 "U2" H 3850 2750 50  0000 C CNN
+F 0 "C" H 3850 2750 50  0000 C CNN
 F 1 "CBUS" H 3900 2650 50  0000 C CNN
 F 2 "Connector_PinHeader_2.54mm:PinHeader_1x08_P2.54mm_Vertical" H 3375 3425 50  0001 C CNN
@@
 	6350 2450 7850 2450
 $Comp
-L FTDI:ABUS U4
+L FTDI:ABUS A
 U 1 1 5F56E993
 P 8100 2750
-F 0 "U4" H 8550 2750 50  0000 C CNN
+F 0 "A" H 8500 2750 50  0000 L CNN
 F 1 "ABUS" H 8600 2650 50  0000 C CNN
 F 2 "Connector_PinHeader_2.54mm:PinHeader_1x08_P2.54mm_Vertical" H 8075 3425 50  0001 C CNN
@@
 $EndComp
 $Comp
-L FTDI:BBUS U5
+L FTDI:BBUS B
 U 1 1 5F51EDE5
 P 8100 3800
-F 0 "U5" H 8478 3801 50  0000 L CNN
+F 0 "B" H 8478 3801 50  0000 L CNN
 F 1 "BBUS" H 8478 3710 50  0000 L CNN
 F 2 "Connector_PinHeader_2.54mm:PinHeader_1x08_P2.54mm_Vertical" H 8075 4475 50  0001 C CNN

Commit message: Restore lost pin
Parts:
- D1, D2, D3, D4, D5, D6, D7, D8: footprint LED_SMD:LED_0805_2012Metric -> neon_footprints:LED_0805_2012Metric
- renumbered A to A1, B to B1, C to C1, D to D9
Changed lines of the file:
@@
 $EndDescr
 $Comp
-L FTDI:DBUS D
+L FTDI:DBUS D9
 U 1 1 5F52AE75
 P 3400 3800
-F 0 "D" H 3850 3800 50  0000 C CNN
+F 0 "D9" H 3850 3800 50  0000 C CNN
 F 1 "DBUS" H 3900 3700 50  0000 C CNN
 F 2 "Connector_PinHeader_2.54mm:PinHeader_1x08_P2.54mm_Vertical" H 3375 4475 50  0001 C CNN
@@
 	5150 2650 3600 2650
 $Comp
-L FTDI:CBUS C
+L FTDI:CBUS C1
 U 1 1 5F520AE1
 P 3400 2750
-F 0 "C" H 3850 2750 50  0000 C CNN
+F 0 "C1" H 3850 2750 50  0000 C CNN
 F 1 "CBUS" H 3900 2650 50  0000 C CNN
 F 2 "Connector_PinHeader_2.54mm:PinHeader_1x08_P2.54mm_Vertical" H 3375 3425 50  0001 C CNN
@@
 F 0 "D6" H 9043 1967 50  0000 C CNN
 F 1 "LED" H 9043 1876 50  0000 C CNN
-F 2 "LED_SMD:LED_0805_2012Metric" H 9050 1750 50  0001 C CNN
+F 2 "neon_footprints:LED_0805_2012Metric" H 9050 1750 50  0001 C CNN
 F 3 "~" H 9050 1750 50  0001 C CNN
 	1    9050 1750
@@
 F 0 "D5" H 9043 1217 50  0000 C CNN
 F 1 "LED" H 9043 1126 50  0000 C CNN
-F 2 "LED_SMD:LED_0805_2012Metric" H 9050 1000 50  0001 C CNN
+F 2 "neon_footprints:LED_0805_2012Metric" H 9050 1000 50  0001 C CNN
 F 3 "~" H 9050 1000 50  0001 C CNN
 	1    9050 1000
@@
 F 0 "D2" H 2443 1967 50  0000 C CNN
 F 1 "LED" H 2443 1876 50  0000 C CNN
-F 2 "LED_SMD:LED_0805_2012Metric" H 2450 1750 50  0001 C CNN
+F 2 "neon_footprints:LED_0805_2012Metric" H 2450 1750 50  0001 C CNN
 F 3 "~" H 2450 1750 50  0001 C CNN
 	1    2450 1750
@@
 F 0 "D1" H 2443 1217 50  0000 C CNN
 F 1 "LED" H 2443 1126 50  0000 C CNN
-F 2 "LED_SMD:LED_0805_2012Metric" H 2450 1000 50  0001 C CNN
+F 2 "neon_footprints:LED_0805_2012Metric" H 2450 1000 50  0001 C CNN
 F 3 "~" H 2450 1000 50  0001 C CNN
 	1    2450 1000
@@
 F 0 "D3" H 2443 5117 50  0000 C CNN
 F 1 "LED" H 2443 5026 50  0000 C CNN
-F 2 "LED_SMD:LED_0805_2012Metric" H 2450 4900 50  0001 C CNN
+F 2 "neon_footprints:LED_0805_2012Metric" H 2450 4900 50  0001 C CNN
 F 3 "~" H 2450 4900 50  0001 C CNN
 	1    2450 4900
@@
 F 0 "D4" H 2443 5867 50  0000 C CNN
 F 1 "LED" H 2443 5776 50  0000 C CNN
-F 2 "LED_SMD:LED_0805_2012Metric" H 2450 5650 50  0001 C CNN
+F 2 "neon_footprints:LED_0805_2012Metric" H 2450 5650 50  0001 C CNN
 F 3 "~" H 2450 5650 50  0001 C CNN
 	1    2450 5650
@@
 	6350 2450 7850 2450
 $Comp
-L FTDI:ABUS A
+L FTDI:ABUS A1
 U 1 1 5F56E993
 P 8100 2750
-F 0 "A" H 8500 2750 50  0000 L CNN
+F 0 "A1" H 8500 2750 50  0000 L CNN
 F 1 "ABUS" H 8600 2650 50  0000 C CNN
 F 2 "Connector_PinHeader_2.54mm:PinHeader_1x08_P2.54mm_Vertical" H 8075 3425 50  0001 C CNN
@@
 $EndComp
 $Comp
-L FTDI:BBUS B
+L FTDI:BBUS B1
 U 1 1 5F51EDE5
 P 8100 3800
-F 0 "B" H 8478 3801 50  0000 L CNN
+F 0 "B1" H 8478 3801 50  0000 L CNN
 F 1 "BBUS" H 8478 3710 50  0000 L CNN
 F 2 "Connector_PinHeader_2.54mm:PinHeader_1x08_P2.54mm_Vertical" H 8075 4475 50  0001 C CNN
@@
 F 0 "D8" H 9043 5867 50  0000 C CNN
 F 1 "LED" H 9043 5776 50  0000 C CNN
-F 2 "LED_SMD:LED_0805_2012Metric" H 9050 5650 50  0001 C CNN
+F 2 "neon_footprints:LED_0805_2012Metric" H 9050 5650 50  0001 C CNN
 F 3 "~" H 9050 5650 50  0001 C CNN
 	1    9050 5650
@@
 F 0 "D7" H 9043 5117 50  0000 C CNN
 F 1 "LED" H 9043 5026 50  0000 C CNN
-F 2 "LED_SMD:LED_0805_2012Metric" H 9050 4900 50  0001 C CNN
+F 2 "neon_footprints:LED_0805_2012Metric" H 9050 4900 50  0001 C CNN
 F 3 "~" H 9050 4900 50  0001 C CNN
 	1    9050 4900

Commit message: With transistors
Parts:
- renumbered J5 to J1, J4 to J2, J2 to J3, J3 to J4, J1 to J5, A1 to U2, B1 to U3, C1 to U4, D9 to U5
Changed lines of the file:
@@
 $EndDescr
 $Comp
-L FTDI:DBUS D9
+L FTDI:DBUS U5
 U 1 1 5F52AE75
 P 3400 3800
-F 0 "D9" H 3850 3800 50  0000 C CNN
+F 0 "U5" H 3850 3800 50  0000 C CNN
 F 1 "DBUS" H 3900 3700 50  0000 C CNN
 F 2 "Connector_PinHeader_2.54mm:PinHeader_1x08_P2.54mm_Vertical" H 3375 4475 50  0001 C CNN
@@
 V3V3
 $Comp
-L FTDI:V3V3-GND J2
+L FTDI:V3V3-GND J3
 U 1 1 5F4D75A0
 P 5600 5300
-F 0 "J2" V 5800 5150 50  0000 L CNN
+F 0 "J3" V 5800 5150 50  0000 L CNN
 F 1 "V3V3-GND" H 5600 5100 50  0001 C CNN
 F 2 "Connector_PinHeader_2.54mm:PinHeader_1x02_P2.54mm_Vertical" H 5600 5300 50  0001 C CNN
@@
 V3V3
 $Comp
-L FTDI:V3V3-GND J3
+L FTDI:V3V3-GND J4
 U 1 1 5F4F496F
 P 5600 5750
-F 0 "J3" V 5800 5600 50  0000 L CNN
+F 0 "J4" V 5800 5600 50  0000 L CNN
 F 1 "V3V3-GND" H 5600 5550 50  0001 C CNN
 F 2 "Connector_PinHeader_2.54mm:PinHeader_1x02_P2.54mm_Vertical" H 5600 5750 50  0001 C CNN
@@
 V3V3
 $Comp
-L FTDI:V3V3-GND J4
+L FTDI:V3V3-GND J2
 U 1 1 5F4F5A0D
 P 5600 6200
-F 0 "J4" V 5800 6050 50  0000 L CNN
+F 0 "J2" V 5800 6050 50  0000 L CNN
 F 1 "V3V3-GND" H 5600 6000 50  0001 C CNN
 F 2 "Connector_PinHeader_2.54mm:PinHeader_1x02_P2.54mm_Vertical" H 5600 6200 50  0001 C CNN
@@
 V3V3
 $Comp
-L FTDI:VBUS-VCC J1
+L FTDI:VBUS-VCC J5
 U 1 1 5F51B746
 P 4500 4650
-F 0 "J1" H 4550 4750 50  0000 L CNN
+F 0 "J5" H 4550 4750 50  0000 L CNN
 F 1 "VBUS-VCC" H 4650 4450 50  0001 C CNN
 F 2 "Connector_PinHeader_2.54mm:PinHeader_1x02_P2.54mm_Vertical" H 4500 4650 50  0001 C CNN
@@
 	5150 2650 3600 2650
 $Comp
-L FTDI:CBUS C1
+L FTDI:CBUS U4
 U 1 1 5F520AE1
 P 3400 2750
-F 0 "C1" H 3850 2750 50  0000 C CNN
+F 0 "U4" H 3900 2750 50  0000 R CNN
 F 1 "CBUS" H 3900 2650 50  0000 C CNN
 F 2 "Connector_PinHeader_2.54mm:PinHeader_1x08_P2.54mm_Vertical" H 3375 3425 50  0001 C CNN
@@
 	6650 4650 6350 4650
 $Comp
-L FTDI:V3V3-VIO J5
+L FTDI:V3V3-VIO J1
 U 1 1 5F4B4881
 P 6950 4650
-F 0 "J5" H 6850 4750 50  0000 L CNN
+F 0 "J1" H 6850 4750 50  0000 L CNN
 F 1 "V3V3-VIO" H 6950 4450 50  0001 C CNN
 F 2 "Connector_PinHeader_2.54mm:PinHeader_1x02_P2.54mm_Vertical" H 6950 4650 50  0001 C CNN
@@
 	6350 2450 7850 2450
 $Comp
-L FTDI:ABUS A1
+L FTDI:ABUS U2
 U 1 1 5F56E993
 P 8100 2750
-F 0 "A1" H 8500 2750 50  0000 L CNN
+F 0 "U2" H 8500 2750 50  0000 L CNN
 F 1 "ABUS" H 8600 2650 50  0000 C CNN
 F 2 "Connector_PinHeader_2.54mm:PinHeader_1x08_P2.54mm_Vertical" H 8075 3425 50  0001 C CNN
@@
 $EndComp
 $Comp
-L FTDI:BBUS B1
+L FTDI:BBUS U3
 U 1 1 5F51EDE5
 P 8100 3800
-F 0 "B1" H 8478 3801 50  0000 L CNN
+F 0 "U3" H 8478 3801 50  0000 L CNN
 F 1 "BBUS" H 8478 3710 50  0000 L CNN
 F 2 "Connector_PinHeader_2.54mm:PinHeader_1x08_P2.54mm_Vertical" H 8075 4475 50  0001 C CNN
