File: neon/neon.kicad_pcb (KiCad board)
At the start: 2 copper layers, 54.7 x 55 mm, 27 parts, among them J1 V3V3-VIO, J2 V3V3-GND, J3 V3V3-GND, J4 V3V3-GND, J5 VBUS-VCC, U1 FT4232H_module, U2 A, U3 B, U4 C, U5 D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

Commit message: With table and LEDs underneath the ftdi
Parts:
- U2: value A -> ABUS
- U3: value B -> BBUS
- U4 (x2): value C -> CBUS
- U5: value D -> DBUS
- moved D5 35.4 mm to (160.1, 94.0)
- moved D6 31.2 mm to (160.0, 91.4)
- moved D1 29.5 mm to (154.9, 118.1), turned to 180 degrees
- moved D2 27.4 mm to (154.9, 115.6), turned to 180 degrees
- moved D3 12.8 mm to (160.7, 118.1), turned to 0 degrees
- moved D4 10.7 mm to (160.7, 115.6)
- moved REF** 9.44 mm to (171.4, 83.8)
- moved REF** 8.54 mm to (171.4, 125.7)
- moved D7 7.10 mm to (154.9, 91.4), turned to 180 degrees
- moved D8 6.87 mm to (154.9, 94.0), turned to 180 degrees
- moved J1 2.54 mm to (170.9, 113.2)
- moved J2 2.54 mm to (170.9, 108.7)
- moved J3 2.54 mm to (170.9, 104.3)
- moved J4 2.54 mm to (170.9, 99.8)
- moved J5 2.54 mm to (170.8, 95.2)
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Routing:
- net V3V3: track 84.6 -> 41.2 mm, vias 2 -> 0
- net GND: track 12.4 -> 4.19 mm
- net Net-(D4-Pad2): track 21.4 -> 25.7 mm
Other:
- board size 54.7 x 55 mm -> 60 x 50 mm
- board text added: "A & B ONLY"
- board text added: "ARX"
- board text added: "ATX"
- board text added: "BRX"
- board text added: "BTX"
- board text added: "CRX"
- board text added: "CTX"
- board text added: "DRX"
- board text added: "DTX"
- board text removed: "GPIO"

Commit message: Sniffer PCB - draft
Parts:
- removed REF** (x4): MountingHole_3.2mm_M3, MountingHole:MountingHole_3.2mm_M3
- removed the U4 at (125.7, 87.6)
- added H1: MountingHole, MountingHole:MountingHole_3.2mm_M3, F.Cu at (119.4, 83.8)
- added H2: MountingHole, MountingHole:MountingHole_3.2mm_M3, F.Cu at (170.8, 83.8)
- added H3: MountingHole, MountingHole:MountingHole_3.2mm_M3, F.Cu at (119.4, 125.7)
- added H4: MountingHole, MountingHole:MountingHole_3.2mm_M3, F.Cu at (171.4, 125.7)
- added S1: sniffer, neon_footprints:PinHeader_1x08_P2.54mm_Vertical, F.Cu at (148.0, 87.5)
- added S2: sniffer, neon_footprints:PinHeader_1x08_P2.54mm_Vertical, F.Cu at (125.7, 87.5)
- added S3: sniffer, neon_footprints:PinHeader_1x08_P2.54mm_Vertical, F.Cu at (177.5, 81.2)
- added S4: sniffer, neon_footprints:PinHeader_1x08_P2.54mm_Vertical, F.Cu at (182.1, 81.2)
- U2: value ABUS -> A
- U3: value BBUS -> B
- U4: value CBUS -> C
- U5: value DBUS -> D
- moved U4 22.2 mm to (148.0, 84.7)
- moved U5 22.2 mm to (125.7, 84.7)
- moved D1 0.64 mm to (154.9, 117.5)
- moved D3 0.64 mm to (160.7, 117.5)
- moved D6 0.64 mm to (160.0, 92.1)
- moved D7 0.64 mm to (154.9, 92.1)
- moved D2 0.63 mm to (154.9, 114.9)
- moved D4 0.63 mm to (160.7, 114.9)
- moved D5 0.63 mm to (160.1, 94.6)
- moved D8 0.63 mm to (154.9, 94.6)
Connections:
- U1 pad 11: Net-(U1-Pad11) -> (no net)
- U1 pad 13: Net-(U1-Pad13) -> (no net)
- U1 pad 14: Net-(U1-Pad14) -> (no net)
- U1 pad 15: Net-(U1-Pad15) -> (no net)
- U1 pad 16: Net-(U1-Pad16) -> (no net)
- U1 pad 17: Net-(U1-Pad17) -> (no net)
- U1 pad 2: Net-(U1-Pad2) -> (no net)
- U1 pad 3: Net-(U1-Pad3) -> (no net)
- U1 pad 41: Net-(U1-Pad41) -> (no net)
- U1 pad 45: Net-(U1-Pad45) -> (no net)
- U1 pad 50: Net-(U1-Pad50) -> (no net)
- U6 pad 9: Net-(U6-Pad9) -> (no net)
