File: neon/neon.kicad_pcb (KiCad board)
At the start: 2 copper layers, 60 x 50 mm, 31 parts, among them J1 V3V3-VIO, J2 3xV3V3-GND, J5 VBUS-VCC, U1 FT4232H_module, U2 C, U3 B, U4 A, U5 D, U6 74HC595

Commit message: Small fixes
Parts:
- moved RN1 0.89 mm to (139.7, 107.4)
- moved RN2 0.89 mm to (139.7, 102.4)
Routing:
- net Net-(RN1-Pad7): track 3.30 -> 0.00 mm
- net Net-(RN2-Pad8): track 2.72 -> 0.00 mm
- net Net-(RN2-Pad7): track 2.53 -> 0.00 mm
- net Net-(RN2-Pad5): track 2.41 -> 0.00 mm
- net Net-(RN2-Pad6): track 2.34 -> 0.21 mm
- net Net-(RN1-Pad6): track 2.34 -> 0.21 mm
- net Net-(RN1-Pad5): track 2.41 -> 0.46 mm
- net Net-(D3-Pad2): track 1.15 -> 0.00 mm
- net Net-(D4-Pad2): track 0.81 -> 0.00 mm
- net Net-(D2-Pad2): track 0.77 -> 0.00 mm
- net Net-(D1-Pad2): track 0.53 -> 0.00 mm
Changed lines of the file:
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@@
     (thickness 1.6)
     (drawings 138)
-    (tracks 21)
+    (tracks 5)
     (zones 0)
     (modules 31)
@@
   )
   (module Resistor_SMD:R_Array_Convex_4x0603 (layer F.Cu)
-    (at 139.7 108.331 180)
+    (at 139.7 107.442 180)
     (descr "Chip Resistor Network, ROHM MNR14 (see mnr_g.pdf)")
     (tags "resistor array")
@@
   )
   (module Resistor_SMD:R_Array_Convex_4x0603 (layer F.Cu)
-    (at 139.7 103.251 180)
+    (at 139.7 102.362 180)
     (descr "Chip Resistor Network, ROHM MNR14 (see mnr_g.pdf)")
     (tags "resistor array")
@@
   )
   (dimension 25 (width 0.15) (layer Dwgs.User)
-    (gr_text "25.000 mm" (at 212.50481 92.43 270) (layer Dwgs.User)
-      (effects (font (size 1 1) (thickness 0.15)))
-    )
-    (feature1 (pts (xy 121.205 104.93) (xy 211.791231 104.93)))
-    (feature2 (pts (xy 121.205 79.93) (xy 211.791231 79.93)))
-    (crossbar (pts (xy 211.20481 79.93) (xy 211.20481 104.93)))
-    (arrow1a (pts (xy 211.20481 104.93) (xy 210.618389 103.803496)))
-    (arrow1b (pts (xy 211.20481 104.93) (xy 211.791231 103.803496)))
-    (arrow2a (pts (xy 211.20481 79.93) (xy 210.618389 81.056504)))
-    (arrow2b (pts (xy 211.20481 79.93) (xy 211.791231 81.056504)))
+    (gr_text "25.000 mm" (at 212.50481 91.541 270) (layer Dwgs.User)
+      (effects (font (size 1 1) (thickness 0.15)))
+    )
+    (feature1 (pts (xy 121.205 104.041) (xy 211.791231 104.041)))
+    (feature2 (pts (xy 121.205 79.041) (xy 211.791231 79.041)))
+    (crossbar (pts (xy 211.20481 79.041) (xy 211.20481 104.041)))
+    (arrow1a (pts (xy 211.20481 104.041) (xy 210.618389 102.914496)))
+    (arrow1b (pts (xy 211.20481 104.041) (xy 211.791231 102.914496)))
+    (arrow2a (pts (xy 211.20481 79.041) (xy 210.618389 80.167504)))
+    (arrow2b (pts (xy 211.20481 79.041) (xy 211.791231 80.167504)))
   )
   (gr_text TX (at 148.59 82.931 90) (layer F.SilkS)
@@
   (gr_line (start 115.49 129.93) (end 175.49 129.93) (layer Edge.Cuts) (width 0.05))
   (gr_line (start 175.49 79.93) (end 175.49 129.93) (layer Edge.Cuts) (width 0.05))
-  (gr_line (start 165.481 101.981) (end 155.321 101.981) (layer F.SilkS) (width 0.12))
+  (gr_line (start 165.354 101.981) (end 155.321 101.981) (layer F.SilkS) (width 0.12))
   (gr_line (start 165.354 111.633) (end 155.194 111.633) (layer F.SilkS) (width 0.12))
   (gr_line (start 165.354 111.3155) (end 165.354 110.6805) (layer F.SilkS) (width 0.12))
@@
   )
   (gr_line (start 115.49 129.93) (end 115.49 79.93) (layer Edge.Cuts) (width 0.05))
-  (segment (start 140.6 109.531) (end 141.127 109.531) (width 0.127) (layer F.Cu) (net 1))
-  (segment (start 141.37 108.731) (end 140.6 108.731) (width 0.127) (layer F.Cu) (net 2))
-  (segment (start 141.751 107.931) (end 140.6 107.931) (width 0.127) (layer F.Cu) (net 3))
-  (segment (start 140.6 107.131) (end 141.408 107.131) (width 0.127) (layer F.Cu) (net 4))
   (segment (start 163.83 113.1151) (end 163.83 113.1151) (width 0.127) (layer F.Cu) (net 10))
   (segment (start 131.564224 108.087776) (end 131.575 108.077) (width 0.127) (layer F.Cu) (net 50))
-  (segment (start 136.849 102.051) (end 136.525 101.727) (width 0.127) (layer F.Cu) (net 51))
-  (segment (start 138.8 102.051) (end 136.849 102.051) (width 0.127) (layer F.Cu) (net 51))
   (segment (start 136.671 102.851) (end 136.525 102.997) (width 0.127) (layer F.Cu) (net 52))
-  (segment (start 138.8 102.851) (end 136.671 102.851) (width 0.127) (layer F.Cu) (net 52))
-  (segment (start 137.141 103.651) (end 136.525 104.267) (width 0.127) (layer F.Cu) (net 53))
-  (segment (start 138.8 103.651) (end 137.141 103.651) (width 0.127) (layer F.Cu) (net 53))
-  (segment (start 137.714 105.537) (end 136.525 105.537) (width 0.127) (layer F.Cu) (net 54))
-  (segment (start 138.8 104.451) (end 137.714 105.537) (width 0.127) (layer F.Cu) (net 54))
   (segment (start 136.849 107.131) (end 136.525 106.807) (width 0.127) (layer F.Cu) (net 55))
-  (segment (start 138.8 107.131) (end 136.849 107.131) (width 0.127) (layer F.Cu) (net 55))
   (segment (start 136.671 107.931) (end 136.525 108.077) (width 0.127) (layer F.Cu) (net 56))
-  (segment (start 138.8 107.931) (end 136.671 107.931) (width 0.127) (layer F.Cu) (net 56))
-  (segment (start 138.8 108.731) (end 138.03 108.731) (width 0.127) (layer F.Cu) (net 57))
-  (segment (start 137.141 108.731) (end 136.525 109.347) (width 0.127) (layer F.Cu) (net 57))
-  (segment (start 138.8 108.731) (end 137.141 108.731) (width 0.127) (layer F.Cu) (net 57))
 )
